File: battle-keeb.kicad_pcb (KiCad board)
At the start: 2 copper layers, 61 parts, among them J1 Conn_01x06_Male, J2 USB_C_Receptacle_USB2.0, SW1 SW_Push, SW2 Rotary_Encoder_Switch, SW3 Rotary_Encoder_Switch, SW4 Rotary_Encoder_Switch, U1 ATmega32U4-AU, Y1 16MHz

Commit message: Placement and Schematic Update
Fixed USB-C Connector on schematic and layout - wurth connector for hand assembly. Placed and adjusted components for control, EMI/EMC, USB, JTAG, and other components.
Parts:
- removed J2: USB_C_Receptacle_USB2.0, Type-C:HRO-TYPE-C-31-M-12
- added USB1: Wurth-632723300011, Type-C:Wurth-632723300011-HandSoldering, F.Cu at (141.3, 63.5)
- D10, D11, D12, D13, D14, D15, D16, D5, D6, D7, D8, D9, FB2: moved to B.Cu
- moved H2 193.5 mm to (173.0, 118.3)
- moved H1 154.6 mm to (173.8, 66.7)
- moved H3 134.1 mm to (219.9, 36.5)
- moved H4 134.1 mm to (228.6, 47.6)
- moved MX1 134.1 mm to (59.5, 73.8)
- moved MX2 134.1 mm to (59.5, 92.9)
- moved MX3 134.1 mm to (59.5, 111.9)
- moved MX4 134.1 mm to (78.6, 73.8)
- moved MX5 134.1 mm to (78.6, 92.9)
- moved MX6 134.1 mm to (78.6, 111.9)
- moved MX7 134.1 mm to (97.6, 73.8)
- moved MX8 134.1 mm to (97.6, 92.9)
- moved MX9 134.1 mm to (97.6, 111.9)
- moved SW2 134.1 mm to (121.4, 71.4)
- moved SW3 134.1 mm to (121.4, 90.5)
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